Commit message: Update common_properties.xacro

File: Armo_description/urdf/common_properties.xacro (robot description, xacro)
@@ -1,5 +1,5 @@
 <?xml version="1.0"?>
 <robot xmlns:xacro="http://www.ros.org/wiki/xacro" >
-    <material name="blck">
+    <material name="black">
         <color rgba="1 1 1 1"/>
     </material>
