Commit message: Update base_mobile.xacro

File: Armo_description/urdf/base_mobile.xacro (robot description, xacro)
@@ -1,5 +1,5 @@
 <?xml version="1.0"?>
 <robot xmlns:xacro="http://www.ros.org/wiki/xacro" >
-    <xacro:property name="base_length" value="0.6"/>
+    <xacro:property name="base_length" value="0.4"/>
     <xacro:property name="base_width" value="0.4"/>
     <xacro:property name="base_height" value="0.2"/>
