Commit message: Update base_mobile_3.xacro

File: Armo_description/urdf/base_mobile_3.xacro (robot description, xacro)
@@ -106,9 +106,9 @@
                 <cylinder radius="0.02" length="0.01"/>
             </geometry>
-            <origin xyz="0 0 -0.005" rpy="0 0 0"/>
+            <origin xyz="0 0 -0.005" rpy="0 ${pi/2.0} 0"/>
             <material name="black"/>
         </visual>
-        <xacro:cylinder_inertia m="0.02" r="0.03" l="0.01" o_xyz="0 0 -0.005" o_rpy="0 0 0"/>
-        <xacro:cylinder_collision r="0.03" l="0.01" o_xyz="0 0 -0.005" o_rpy="0 0 0"/>
+        <xacro:cylinder_inertia m="0.02" r="0.03" l="0.01" o_xyz="0 0 -0.005" o_rpy="0 ${pi/2.0} 0"/>
+        <xacro:cylinder_collision r="0.03" l="0.01" o_xyz="0 0 -0.005" o_rpy="0 ${pi/2.0} 0"/>
     </link>
     <joint name="base_footprint_base_joint" type="fixed">
@@ -165,5 +165,5 @@
         <parent link="camera_link"/>
         <child link="optical_camera_link"/>
-        <origin xyz="${camera_length*1.5} 0 0" rpy="0 ${pi/2} 0"/>
+        <origin xyz="${camera_length*1.5} 0 0" rpy="0 0 0"/>
     </joint>
     <xacro:cube_link prefix="scan" m="1.2" l="0.1" b="0.1" h="0.1" x="0" y="0" z="0.05" r="0" p="0" yaw="0"/>
